File: Circuit/Reference/Reference Driver/Reference.sch (EAGLE design)
At the start: 11 parts

Commit message: Add the mosfets and their driver to the BLDC Driver sch
Parts:
- C2, C3, C4, C5, C6, C7, C8, C9: device rcl:C-USC0805 -> rcl:C-USC0603
- R1, R2: device rcl:R-US_M0805 -> rcl:R-US_R0603
