File: Circuit/V3/Driver.sch (EAGLE design)
At the start: 35 parts, among them IC1 DRV8303DCA

Commit message: Fixed some bugs and edited the note.md
Parts:
- removed R3: 1, SparkFun-Resistors:1OHM-0603-1/10W-1%
- added C16: 2.2nF, SparkFun-Capacitors:2.2NF/2200PF-0603-50V-10%
- added R5, R7: 0, SparkFun-Resistors:0OHM-0603-1/10W
Connections:
- removed net N$26: IC1.DTC, R3.2
- new net N$1: IC1.SO1, R5.2
- net GND: now also C16.2, IC1.DTC; no longer R3.1
- net N$3: now also IC1.SO2, R7.2; no longer U$1.3.3V
- net PB0: now also C16.1, R7.1; no longer IC1.SO2
- net PB1: now also R5.1; no longer IC1.SO1
- net VCC: now also U$1.3.3V; no longer U$1.5V
Changed lines of the file:
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@@
 <part name="P+2" library="supply1" library_urn="urn:adsk.eagle:library:371" deviceset="VCC" device=""/>
 <part name="C1" library="SparkFun-Capacitors" deviceset="0.1UF" device="-0603-25V-(+80/-20%)" value="0.1uF"/>
-<part name="R3" library="SparkFun-Resistors" deviceset="1OHM" device="-0603-1/10W-1%" value="1"/>
 <part name="SUPPLY2" library="supply2" library_urn="urn:adsk.eagle:library:372" deviceset="GND" device=""/>
 <part name="R4" library="SparkFun-Resistors" deviceset="10KOHM" device="-0603-1/10W-1%" value="10k"/>
@@
 <part name="SUPPLY22" library="supply2" library_urn="urn:adsk.eagle:library:372" deviceset="GND" device=""/>
 <part name="SUPPLY23" library="supply2" library_urn="urn:adsk.eagle:library:372" deviceset="GND" device=""/>
+<part name="R5" library="SparkFun-Resistors" deviceset="0OHM" device="-0603-1/10W" value="0"/>
+<part name="R7" library="SparkFun-Resistors" deviceset="0OHM" device="-0603-1/10W" value="0"/>
+<part name="SUPPLY24" library="supply2" library_urn="urn:adsk.eagle:library:372" deviceset="GND" device=""/>
+<part name="C16" library="SparkFun-Capacitors" deviceset="2.2NF/2200PF" device="-0603-50V-10%" value="2.2nF"/>
 </parts>
 <sheets>
@@
 <attribute name="VALUE" x="27.305" y="85.725" size="1.778" layer="96" rot="R270"/>
 </instance>
-<instance part="P+1" gate="VCC" x="20.32" y="86.36" smashed="yes" rot="R90">
-<attribute name="VALUE" x="22.86" y="83.82" size="1.778" layer="96" rot="R180"/>
+<instance part="P+1" gate="VCC" x="91.44" y="124.46" smashed="yes" rot="R270">
+<attribute name="VALUE" x="93.98" y="121.92" size="1.778" layer="96"/>
 </instance>
 <instance part="SUPPLY8" gate="GND" x="170.18" y="15.24" smashed="yes">
@@
 <attribute name="VALUE" x="271.399" y="141.224" size="1.778" layer="96" font="vector" rot="R90"/>
 </instance>
-<instance part="R3" gate="G$1" x="203.2" y="144.78" smashed="yes">
-<attribute name="NAME" x="203.2" y="146.304" size="1.778" layer="95" font="vector" align="bottom-center"/>
-<attribute name="VALUE" x="203.2" y="143.256" size="1.778" layer="96" font="vector" align="top-center"/>
-</instance>
 <instance part="SUPPLY2" gate="GND" x="193.04" y="144.78" smashed="yes" rot="R270">
 <attribute name="VALUE" x="189.865" y="146.685" size="1.778" layer="96" rot="R270"/>
@@
 <instance part="SUPPLY23" gate="GND" x="193.04" y="114.3" smashed="yes" rot="R270">
 <attribute name="VALUE" x="189.865" y="116.205" size="1.778" layer="96" rot="R270"/>
+</instance>
+<instance part="R5" gate="G$1" x="200.66" y="99.06" smashed="yes">
+<attribute name="NAME" x="198.12" y="100.584" size="1.778" layer="95" font="vector" align="bottom-center"/>
+</instance>
+<instance part="R7" gate="G$1" x="200.66" y="96.52" smashed="yes">
+<attribute name="NAME" x="200.66" y="92.964" size="1.778" layer="95" font="vector" align="bottom-center"/>
+</instance>
+<instance part="SUPPLY24" gate="GND" x="193.04" y="81.28" smashed="yes">
+<attribute name="VALUE" x="191.135" y="78.105" size="1.778" layer="96"/>
+</instance>
+<instance part="C16" gate="G$1" x="193.04" y="88.9" smashed="yes">
+<attribute name="NAME" x="194.564" y="91.821" size="1.778" layer="95" font="vector"/>
+<attribute name="VALUE" x="194.564" y="86.741" size="1.778" layer="96" font="vector"/>
 </instance>
 </instances>
@@
 </segment>
 <segment>
-<pinref part="R3" gate="G$1" pin="1"/>
 <pinref part="SUPPLY2" gate="GND" pin="GND"/>
-<wire x1="195.58" y1="144.78" x2="198.12" y2="144.78" width="0.1524" layer="91"/>
+<pinref part="IC1" gate="G$1" pin="DTC"/>
+<wire x1="195.58" y1="144.78" x2="215.9" y2="144.78" width="0.1524" layer="91"/>
 </segment>
 <segment>
@@
 <pinref part="SUPPLY23" gate="GND" pin="GND"/>
 </segment>
-</net>
-<net name="N$3" class="0">
-<segment>
-<pinref part="U$1" gate="G$1" pin="3.3V"/>
-<wire x1="78.74" y1="124.46" x2="83.82" y2="124.46" width="0.1524" layer="91"/>
+<segment>
+<pinref part="SUPPLY24" gate="GND" pin="GND"/>
+<wire x1="193.04" y1="83.82" x2="193.04" y2="86.36" width="0.1524" layer="91"/>
+<pinref part="C16" gate="G$1" pin="2"/>
 </segment>
 </net>
@@
 </segment>
 <segment>
-<pinref part="IC1" gate="G$1" pin="SO1"/>
-<wire x1="215.9" y1="99.06" x2="213.36" y2="99.06" width="0.1524" layer="91"/>
-<label x="213.36" y="99.06" size="1.27" layer="95" rot="R180" xref="yes"/>
+<pinref part="R5" gate="G$1" pin="1"/>
+<wire x1="195.58" y1="99.06" x2="190.5" y2="99.06" width="0.1524" layer="91"/>
+<label x="190.5" y="99.06" size="1.27" layer="95" rot="R180" xref="yes"/>
 </segment>
 </net>
@@
 </segment>
 <segment>
-<pinref part="IC1" gate="G$1" pin="SO2"/>
-<wire x1="215.9" y1="96.52" x2="213.36" y2="96.52" width="0.1524" layer="91"/>
-<label x="213.36" y="96.52" size="1.27" layer="95" rot="R180" xref="yes"/>
+<label x="190.5" y="96.52" size="1.27" layer="95" rot="R180" xref="yes"/>
+<wire x1="193.04" y1="96.52" x2="190.5" y2="96.52" width="0.1524" layer="91"/>
+<wire x1="193.04" y1="96.52" x2="193.04" y2="93.98" width="0.1524" layer="91"/>
+<pinref part="C16" gate="G$1" pin="1"/>
+<pinref part="R7" gate="G$1" pin="1"/>
+<wire x1="195.58" y1="96.52" x2="193.04" y2="96.52" width="0.1524" layer="91"/>
 </segment>
 </net>
@@
 <net name="VCC" class="0">
 <segment>
-<pinref part="U$1" gate="G$1" pin="5V"/>
-<wire x1="38.1" y1="86.36" x2="22.86" y2="86.36" width="0.1524" layer="91"/>
-<pinref part="P+1" gate="VCC" pin="VCC"/>
-</segment>
-<segment>
 <pinref part="5V" gate="B" pin="TP"/>
 <wire x1="0" y1="86.36" x2="2.54" y2="86.36" width="0.1524" layer="91"/>
@@
 <wire x1="215.9" y1="101.6" x2="210.82" y2="101.6" width="0.1524" layer="91"/>
 <pinref part="P+4" gate="VCC" pin="VCC"/>
+</segment>
+<segment>
+<pinref part="U$1" gate="G$1" pin="3.3V"/>
+<wire x1="78.74" y1="124.46" x2="88.9" y2="124.46" width="0.1524" layer="91"/>
+<pinref part="P+1" gate="VCC" pin="VCC"/>
 </segment>
 </net>
@@
 </segment>
 </net>
-<net name="N$26" class="0">
-<segment>
-<pinref part="IC1" gate="G$1" pin="DTC"/>
-<wire x1="215.9" y1="144.78" x2="208.28" y2="144.78" width="0.1524" layer="91"/>
-<pinref part="R3" gate="G$1" pin="2"/>
-</segment>
-</net>
 <net name="N$32" class="0">
 <segment>
@@
 </segment>
 </net>
+<net name="N$1" class="0">
+<segment>
+<pinref part="IC1" gate="G$1" pin="SO1"/>
+<pinref part="R5" gate="G$1" pin="2"/>
+<wire x1="215.9" y1="99.06" x2="205.74" y2="99.06" width="0.1524" layer="91"/>
+</segment>
+</net>
+<net name="N$3" class="0">
+<segment>
+<pinref part="IC1" gate="G$1" pin="SO2"/>
+<pinref part="R7" gate="G$1" pin="2"/>
+<wire x1="215.9" y1="96.52" x2="205.74" y2="96.52" width="0.1524" layer="91"/>
+</segment>
+</net>

Commit message: Fixed some bugs
Changed lines of the file:
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@@
 <pinref part="LC" gate="G$1" pin="S"/>
 <wire x1="312.42" y1="-30.48" x2="312.42" y2="-45.72" width="0.1524" layer="91"/>
+<junction x="312.42" y="-30.48"/>
 </segment>
 <segment>
@@
 <pinref part="SUPPLY10" gate="GND" pin="GND"/>
 <junction x="205.74" y="93.98"/>
+<junction x="215.9" y="91.44"/>
 </segment>
 <segment>
@@
 <wire x1="256.54" y1="83.82" x2="256.54" y2="81.28" width="0.1524" layer="91"/>
 <pinref part="SUPPLY19" gate="GND" pin="GND"/>
+<junction x="256.54" y="83.82"/>
 </segment>
 <segment>
@@
 <pinref part="R7" gate="G$1" pin="1"/>
 <wire x1="195.58" y1="96.52" x2="193.04" y2="96.52" width="0.1524" layer="91"/>
+<junction x="193.04" y="96.52"/>
 </segment>
 </net>
@@
 <wire x1="271.78" y1="109.22" x2="274.32" y2="109.22" width="0.1524" layer="91"/>
 <label x="274.32" y="109.22" size="1.27" layer="95" xref="yes"/>
+<junction x="271.78" y="109.22"/>
 </segment>
 </net>
@@
 <wire x1="271.78" y1="121.92" x2="274.32" y2="121.92" width="0.1524" layer="91"/>
 <label x="274.32" y="121.92" size="1.27" layer="95" xref="yes"/>
+<junction x="271.78" y="121.92"/>
 </segment>
 </net>
@@
 <wire x1="271.78" y1="134.62" x2="274.32" y2="134.62" width="0.1524" layer="91"/>
 <label x="274.32" y="134.62" size="1.27" layer="95" xref="yes"/>
+<junction x="271.78" y="134.62"/>
 </segment>
 </net>
@@
 <pinref part="R6" gate="G$1" pin="2"/>
 <wire x1="200.66" y1="160.02" x2="200.66" y2="157.48" width="0.1524" layer="91"/>
-</segment>
-<segment>
+<junction x="195.58" y="160.02"/>
+</segment>
+<segment>
