File: V1.1/Circuit/Driver.sch (EAGLE design)
At the start: 2 parts, among them IC1 DRV8300DIPWR

Commit message: Added Not Gate to the circuit
Parts:
- added C1: 10uF, SparkFun-Capacitors:10UF-0603-6.3V-20%
- added C2, C3, C4: 1.0uF, SparkFun-Capacitors:1.0UF-0603-16V-10%
- added IC2: CD74HC4049PWR, CD74HC4049PWR:CD74HC4049PWR
- added R1, R2, R3, R4, R5, R6: 100, SparkFun-Resistors:100OHM-0603-1/10W-1%
- added R7, R8, R9: CR2512-FX-51R1ELF, CR2512-FX-51R1ELF:CR2512-FX-51R1ELF
- added TP1: PTR2, testpad:PTR2
- added TP2, TP3, TP4: TPTP20SQ, testpad:TPTP20SQ
- added U$2, U$3, U$4, U$5, U$6, U$7: IRLR7843, BLDC project:IRLR7843
Connections:
- removed net PA10: U$1.PA10
- removed net PA8: U$1.PA8
- removed net PB7: U$1.PB7
- new net BSTA: C2.2, IC1.BSTA
- new net BSTB: C3.2, IC1.BSTB
- new net BSTC: C4.2, IC1.BSTC
- new net GHA: IC1.GHA, R1.1
- new net GHB: IC1.GHB, R2.1
- new net GHC: IC1.GHC, R3.1
- new net GLA: IC1.GLA
- new net GLB: IC1.GLB
- new net GLC: IC1.GLC
- new net INHA: IC1.INHA, IC2.1A, U$1.PA8
- new net INHB: IC1.INHB, IC2.2A, U$1.PA10
- new net INHC: IC1.INHC, IC2.3A, U$1.PB7
- new net INLA: IC1.INLA, IC2.!1Y
- new net INLB: IC1.INLB, IC2.!2Y
- new net INLC: IC1.INLC, IC2.!3Y
- new net N$1: R1.2, U$2.G
- new net N$2: R2.2, U$4.G
- new net N$3: R3.2, U$6.G
- new net N$4: R5.2, U$3.G
- new net N$5: R6.2, U$5.G
- new net N$6: R4.2, U$7.G
- new net N$7: R7.1, TP2.TP
- new net N$8: R8.1, TP3.TP
- new net N$9: R9.1, TP4.TP
- new net SHA: C2.1, IC1.SHA, R5.1, R7.2, U$2.S, U$3.D
- new net SHB: C3.1, IC1.SHB, R6.1, R8.2, U$4.S, U$5.D
- new net SHC: C4.1, IC1.SHC, R4.1, R9.2, U$6.S, U$7.D
- new net VCC: C1.1, IC1.GVDD, TP1-1.TP, U$2.D, U$4.D, U$6.D
- net 3V3: now also IC2.VCC
- net GND: now also C1.2, IC1.GND, IC2.4A, IC2.5A, IC2.6A, IC2.GND, TP1-2.TP, U$3.S, U$5.S, U$7.S

Commit message: Ready for autoroutering
Parts:
- removed TP1: PTR2, testpad:PTR2
- removed TP2, TP3, TP4: TPTP20SQ, testpad:TPTP20SQ
- added A, B, C: (no value), wirepad:SMD5
- added GND, TP6, TP7, VCC: TPPAD1-13Y, testpad:TPPAD1-13Y
- added U1, U2, U3: INA240A1PWR, INA240A1PWR:INA240A1PWR
Connections:
- removed net N$7: R7.1, TP2.TP
- removed net N$8: R8.1, TP3.TP
- removed net N$9: R9.1, TP4.TP
- new net SLA: A.P, R7.1, U1.IN-
- new net SLB: B.P, R8.1, U2.IN-
- new net SLC: C.P, R9.1, U3.IN-
- net 3V3: now also TP6.TP, U1.REF2, U1.VS, U2.REF2, U2.VS, U3.REF2, U3.VS
- net GLA: now also R5.1
- net GLB: now also R6.1
- net GLC: now also R4.1
- net GND: now also GND.TP, TP7.TP, U1.GND, U1.REF1, U2.GND, U2.REF1, U3.GND, U3.REF1; no longer TP1-2.TP
- net PA3: now also U3.OUT
- net PB0: now also U2.OUT
- net PB1: now also U1.OUT
- net SHA: now also U1.IN+; no longer R5.1
- net SHB: now also U2.IN+; no longer R6.1
- net SHC: now also U3.IN+; no longer R4.1
- net VCC: now also VCC.TP; no longer TP1-1.TP
