File: V3-DRV8300/Circuit/Tester.brd (EAGLE design)
At the start: 27.9 x 34.9 mm, 27 parts, among them IC1 DRV8303DCA

Commit message: Ready for autoroutering (Tester) 2
Parts:
- moved AVDD_CAP 0.63 mm to (6.67, 10.8)
- moved C9 0.63 mm to (6.67, 17.5)
- moved DVDD_CAP 0.63 mm to (6.67, 14.1)
Routing:
- net N$47: track 3.13 -> 3.77 mm
- net N$43: track 3.07 -> 3.70 mm
- net N$34: track 3.67 -> 4.31 mm
- net N$33: track 3.18 -> 3.81 mm
- net GND: track 50.8 -> 51.4 mm
Changed lines of the file:
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@@
 </autorouter>
 <elements>
-<element name="AVDD_CAP" library="SparkFun-Capacitors" package="0603" value="1.0uF" x="7.3025" y="10.795" smashed="yes" rot="R270">
-<attribute name="NAME" x="5.842" y="10.4775" size="0.6096" layer="25" font="vector" ratio="20" rot="R270" align="bottom-center"/>
-<attribute name="PROD_ID" value="CAP-00868" x="-9.2075" y="-4.445" size="1.778" layer="27" rot="R270" display="off"/>
-<attribute name="VALUE" x="8.763" y="10.795" size="0.6096" layer="27" font="vector" ratio="20" rot="R270" align="top-center"/>
+<element name="AVDD_CAP" library="SparkFun-Capacitors" package="0603" value="1.0uF" x="6.6675" y="10.795" smashed="yes" rot="R270">
+<attribute name="PROD_ID" value="CAP-00868" x="-9.8425" y="-4.445" size="1.778" layer="27" rot="R270" display="off"/>
+<attribute name="VALUE" x="8.128" y="10.795" size="0.6096" layer="27" font="vector" ratio="20" rot="R270" align="top-center"/>
 </element>
 <element name="C1" library="SparkFun-Capacitors" package="0603" value="0.1uF" x="20.6375" y="22.06625" smashed="yes" rot="R270">
@@
 <attribute name="VALUE" x="7.14375" y="21.082" size="0.6096" layer="27" font="vector" ratio="20" rot="R180" align="top-center"/>
 </element>
-<element name="C9" library="SparkFun-Capacitors" package="0603" value="0.22uF" x="7.3025" y="17.4625" smashed="yes" rot="R90">
-<attribute name="PROD_ID" value="CAP-07822" x="23.8125" y="50.4825" size="1.778" layer="27" rot="R90" display="off"/>
-<attribute name="VALUE" x="8.22325" y="17.4625" size="0.6096" layer="27" font="vector" ratio="20" rot="R90" align="top-center"/>
+<element name="C9" library="SparkFun-Capacitors" package="0603" value="0.22uF" x="6.6675" y="17.4625" smashed="yes" rot="R90">
+<attribute name="PROD_ID" value="CAP-07822" x="23.1775" y="50.4825" size="1.778" layer="27" rot="R90" display="off"/>
+<attribute name="VALUE" x="7.58825" y="17.4625" size="0.6096" layer="27" font="vector" ratio="20" rot="R90" align="top-center"/>
 </element>
 <element name="D1" library="SparkFun-LED" package="LED-0603" value="BLUE" x="23.01875" y="32.385" smashed="yes" rot="R90">
@@
 <attribute name="PROD_ID" value="DIO-08575" x="49.05375" y="47.625" size="1.778" layer="27" rot="R90" display="off"/>
 </element>
-<element name="DVDD_CAP" library="SparkFun-Capacitors" package="0603" value="1.0uF" x="7.3025" y="14.12875" smashed="yes" rot="R90">
-<attribute name="NAME" x="6.5405" y="14.12875" size="0.6096" layer="25" font="vector" ratio="20" rot="R90" align="bottom-center"/>
-<attribute name="PROD_ID" value="CAP-00868" x="23.8125" y="34.44875" size="1.778" layer="27" rot="R90" display="off"/>
-<attribute name="VALUE" x="8.22325" y="14.12875" size="0.6096" layer="27" font="vector" ratio="20" rot="R90" align="top-center"/>
+<element name="DVDD_CAP" library="SparkFun-Capacitors" package="0603" value="1.0uF" x="6.6675" y="14.12875" smashed="yes" rot="R90">
+<attribute name="PROD_ID" value="CAP-00868" x="23.1775" y="34.44875" size="1.778" layer="27" rot="R90" display="off"/>
+<attribute name="VALUE" x="7.58825" y="14.12875" size="0.6096" layer="27" font="vector" ratio="20" rot="R90" align="top-center"/>
 </element>
 <element name="IC1" library="DRV8303DCA" package="SOP50P810X120-49N" value="DRV8303DCA" x="13.97" y="17.78" smashed="yes">
@@
 <contactref element="J8" pad="6"/>
 <contactref element="VIN" pad="1"/>
-<wire x1="10.182" y1="12.03" x2="9.3875" y2="12.03" width="0.3302" layer="1"/>
-<wire x1="9.3875" y1="12.03" x2="7.3025" y2="9.945" width="0.3302" layer="1"/>
+<wire x1="10.182" y1="12.03" x2="8.7525" y2="12.03" width="0.3302" layer="1"/>
+<wire x1="8.7525" y1="12.03" x2="6.6675" y2="9.945" width="0.3302" layer="1"/>
 <polygon width="0.0762" layer="1" spacing="0.000003125" orphans="yes" thermals="no" rank="2">
 <vertex x="11.1125" y="23.8125"/>
@@
 <vertex x="15.5575" y="19.3675"/>
 </polygon>
-<wire x1="6.3961" y1="12.3633375" x2="6.3961" y2="10.9266625" width="0.508" layer="1"/>
-<wire x1="7.3025" y1="13.27875" x2="7.3025" y2="13.2697375" width="0.508" layer="1"/>
-<wire x1="7.3025" y1="10.0202625" x2="7.3025" y2="9.945" width="0.508" layer="1"/>
-<wire x1="7.3025" y1="13.2697375" x2="6.3961" y2="12.3633375" width="0.508" layer="1"/>
-<wire x1="6.3961" y1="10.9266625" x2="7.3025" y2="10.0202625" width="0.508" layer="1"/>
 <wire x1="19.745325" y1="1.40335" x2="18.672175" y2="1.40335" width="0.4064" layer="1"/>
 <wire x1="21.74875" y1="2.69875" x2="21.040725" y2="2.69875" width="0.4064" layer="1"/>
@@
 <wire x1="21.040725" y1="2.69875" x2="19.745325" y2="1.40335" width="0.4064" layer="1"/>
 <wire x1="18.672175" y1="1.40335" x2="17.376775" y2="2.69875" width="0.4064" layer="1"/>
+<wire x1="5.8119" y1="12.34229375" x2="5.8119" y2="10.94770625" width="0.4064" layer="1"/>
+<wire x1="6.6675" y1="13.27875" x2="6.6675" y2="13.19789375" width="0.4064" layer="1"/>
+<wire x1="6.6675" y1="10.09210625" x2="6.6675" y2="9.945" width="0.4064" layer="1"/>
+<wire x1="6.6675" y1="13.19789375" x2="5.8119" y2="12.34229375" width="0.4064" layer="1"/>
+<wire x1="5.8119" y1="10.94770625" x2="6.6675" y2="10.09210625" width="0.4064" layer="1"/>
 <wire x1="21.11375" y1="33.262" x2="23.01875" y2="33.262" width="0" layer="19" extent="1-1"/>
 <wire x1="17.758" y1="23.53" x2="21.11375" y2="33.262" width="0" layer="19" extent="1-1"/>
@@
 <wire x1="6.29375" y1="20.32" x2="10.182" y2="22.53" width="0" layer="19" extent="1-1"/>
 <wire x1="23.1775" y1="11.90625" x2="17.758" y2="12.53" width="0" layer="19" extent="1-1"/>
-<wire x1="6.6675" y1="3.54875" x2="7.3025" y2="9.945" width="0" layer="19" extent="1-1"/>
+<wire x1="6.6675" y1="3.54875" x2="6.6675" y2="9.945" width="0" layer="19" extent="1-1"/>
 </signal>
 <signal name="SO1">
@@
 <contactref element="IC1" pad="10"/>
 <contactref element="C9" pad="2"/>
-<wire x1="7.3025" y1="18.3125" x2="8.02" y2="19.03" width="0.3302" layer="1"/>
-<wire x1="8.02" y1="19.03" x2="10.182" y2="19.03" width="0.3302" layer="1"/>
+<wire x1="6.6675" y1="18.3125" x2="7.385" y2="19.03" width="0.3302" layer="1"/>
+<wire x1="7.385" y1="19.03" x2="10.182" y2="19.03" width="0.3302" layer="1"/>
 </signal>
 <signal name="N$34">
 <contactref element="IC1" pad="11"/>
 <contactref element="C9" pad="1"/>
-<wire x1="7.3025" y1="16.6125" x2="9.22" y2="18.53" width="0.3302" layer="1"/>
-<wire x1="9.22" y1="18.53" x2="10.182" y2="18.53" width="0.3302" layer="1"/>
+<wire x1="6.6675" y1="16.6125" x2="8.585" y2="18.53" width="0.3302" layer="1"/>
+<wire x1="8.585" y1="18.53" x2="10.182" y2="18.53" width="0.3302" layer="1"/>
 </signal>
 <signal name="N$43">
 <contactref element="IC1" pad="19"/>
 <contactref element="DVDD_CAP" pad="2"/>
-<wire x1="10.182" y1="14.53" x2="7.75125" y2="14.53" width="0.381" layer="1"/>
-<wire x1="7.75125" y1="14.53" x2="7.3025" y2="14.97875" width="0.381" layer="1"/>
+<wire x1="10.182" y1="14.53" x2="7.11625" y2="14.53" width="0.381" layer="1"/>
+<wire x1="7.11625" y1="14.53" x2="6.6675" y2="14.97875" width="0.381" layer="1"/>
 </signal>
 <signal name="N$47">
@@
 <contactref element="AVDD_CAP" pad="1"/>
 <wire x1="10.182" y1="12.53" x2="9.36625" y2="12.53" width="0.3302" layer="1"/>
-<wire x1="7.3025" y1="11.645" x2="8.2209" y2="12.5634" width="0.4318" layer="1"/>
-<wire x1="8.2209" y1="12.5634" x2="9.24024375" y2="12.5634" width="0.4318" layer="1"/>
+<wire x1="6.6675" y1="11.645" x2="7.5859" y2="12.5634" width="0.4318" layer="1"/>
+<wire x1="7.5859" y1="12.5634" x2="9.24024375" y2="12.5634" width="0.4318" layer="1"/>
 <wire x1="9.24024375" y1="12.5634" x2="9.36625" y2="12.53" width="0" layer="19" extent="1-1"/>
 </signal>

Commit message: Ready for autoroutering (Tester) 3
Parts:
- moved AVDD_CAP 0.48 mm to (6.19, 10.8)
- moved C9 0.48 mm to (6.19, 17.5)
- moved DVDD_CAP 0.48 mm to (6.19, 14.1)
Changed lines of the file:
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@@
 <param name="RoutingGrid" value="50mil"/>
 <param name="AutoGrid" value="1"/>
-<param name="Efforts" value="0"/>
+<param name="Efforts" value="2"/>
 <param name="TopRouterVariant" value="1"/>
 <param name="tpViaShape" value="round"/>
@@
 </autorouter>
 <elements>
-<element name="AVDD_CAP" library="SparkFun-Capacitors" package="0603" value="1.0uF" x="6.6675" y="10.795" smashed="yes" rot="R270">
-<attribute name="PROD_ID" value="CAP-00868" x="-9.8425" y="-4.445" size="1.778" layer="27" rot="R270" display="off"/>
-<attribute name="VALUE" x="8.128" y="10.795" size="0.6096" layer="27" font="vector" ratio="20" rot="R270" align="top-center"/>
+<element name="AVDD_CAP" library="SparkFun-Capacitors" package="0603" value="1.0uF" x="6.19125" y="10.795" smashed="yes" rot="R270">
+<attribute name="PROD_ID" value="CAP-00868" x="-10.31875" y="-4.445" size="1.778" layer="27" rot="R270" display="off"/>
+<attribute name="VALUE" x="7.65175" y="10.795" size="0.6096" layer="27" font="vector" ratio="20" rot="R270" align="top-center"/>
 </element>
 <element name="C1" library="SparkFun-Capacitors" package="0603" value="0.1uF" x="20.6375" y="22.06625" smashed="yes" rot="R270">
@@
 <attribute name="VALUE" x="7.14375" y="21.082" size="0.6096" layer="27" font="vector" ratio="20" rot="R180" align="top-center"/>
 </element>
-<element name="C9" library="SparkFun-Capacitors" package="0603" value="0.22uF" x="6.6675" y="17.4625" smashed="yes" rot="R90">
-<attribute name="PROD_ID" value="CAP-07822" x="23.1775" y="50.4825" size="1.778" layer="27" rot="R90" display="off"/>
-<attribute name="VALUE" x="7.58825" y="17.4625" size="0.6096" layer="27" font="vector" ratio="20" rot="R90" align="top-center"/>
+<element name="C9" library="SparkFun-Capacitors" package="0603" value="0.22uF" x="6.19125" y="17.4625" smashed="yes" rot="R90">
+<attribute name="PROD_ID" value="CAP-07822" x="22.70125" y="50.4825" size="1.778" layer="27" rot="R90" display="off"/>
+<attribute name="VALUE" x="7.112" y="17.4625" size="0.6096" layer="27" font="vector" ratio="20" rot="R90" align="top-center"/>
 </element>
 <element name="D1" library="SparkFun-LED" package="LED-0603" value="BLUE" x="23.01875" y="32.385" smashed="yes" rot="R90">
@@
 <attribute name="PROD_ID" value="DIO-08575" x="49.05375" y="47.625" size="1.778" layer="27" rot="R90" display="off"/>
 </element>
-<element name="DVDD_CAP" library="SparkFun-Capacitors" package="0603" value="1.0uF" x="6.6675" y="14.12875" smashed="yes" rot="R90">
-<attribute name="PROD_ID" value="CAP-00868" x="23.1775" y="34.44875" size="1.778" layer="27" rot="R90" display="off"/>
-<attribute name="VALUE" x="7.58825" y="14.12875" size="0.6096" layer="27" font="vector" ratio="20" rot="R90" align="top-center"/>
+<element name="DVDD_CAP" library="SparkFun-Capacitors" package="0603" value="1.0uF" x="6.19125" y="14.12875" smashed="yes" rot="R90">
+<attribute name="PROD_ID" value="CAP-00868" x="22.70125" y="34.44875" size="1.778" layer="27" rot="R90" display="off"/>
+<attribute name="VALUE" x="7.112" y="14.12875" size="0.6096" layer="27" font="vector" ratio="20" rot="R90" align="top-center"/>
 </element>
 <element name="IC1" library="DRV8303DCA" package="SOP50P810X120-49N" value="DRV8303DCA" x="13.97" y="17.78" smashed="yes">
@@
 <contactref element="J8" pad="6"/>
 <contactref element="VIN" pad="1"/>
-<wire x1="10.182" y1="12.03" x2="8.7525" y2="12.03" width="0.3302" layer="1"/>
-<wire x1="8.7525" y1="12.03" x2="6.6675" y2="9.945" width="0.3302" layer="1"/>
+<wire x1="10.182" y1="12.03" x2="8.27625" y2="12.03" width="0.3302" layer="1"/>
+<wire x1="8.27625" y1="12.03" x2="6.19125" y2="9.945" width="0.3302" layer="1"/>
 <polygon width="0.0762" layer="1" spacing="0.000003125" orphans="yes" thermals="no" rank="2">
 <vertex x="11.1125" y="23.8125"/>
@@
 <wire x1="21.040725" y1="2.69875" x2="19.745325" y2="1.40335" width="0.4064" layer="1"/>
 <wire x1="18.672175" y1="1.40335" x2="17.376775" y2="2.69875" width="0.4064" layer="1"/>
-<wire x1="5.8119" y1="12.34229375" x2="5.8119" y2="10.94770625" width="0.4064" layer="1"/>
-<wire x1="6.6675" y1="13.27875" x2="6.6675" y2="13.19789375" width="0.4064" layer="1"/>
-<wire x1="6.6675" y1="10.09210625" x2="6.6675" y2="9.945" width="0.4064" layer="1"/>
-<wire x1="6.6675" y1="13.19789375" x2="5.8119" y2="12.34229375" width="0.4064" layer="1"/>
-<wire x1="5.8119" y1="10.94770625" x2="6.6675" y2="10.09210625" width="0.4064" layer="1"/>
+<wire x1="5.33565" y1="12.34229375" x2="5.33565" y2="10.94770625" width="0.4064" layer="1"/>
+<wire x1="6.19125" y1="13.27875" x2="6.19125" y2="13.19789375" width="0.4064" layer="1"/>
+<wire x1="6.19125" y1="10.09210625" x2="6.19125" y2="9.945" width="0.4064" layer="1"/>
+<wire x1="6.19125" y1="13.19789375" x2="5.33565" y2="12.34229375" width="0.4064" layer="1"/>
+<wire x1="5.33565" y1="10.94770625" x2="6.19125" y2="10.09210625" width="0.4064" layer="1"/>
 <wire x1="21.11375" y1="33.262" x2="23.01875" y2="33.262" width="0" layer="19" extent="1-1"/>
 <wire x1="17.758" y1="23.53" x2="21.11375" y2="33.262" width="0" layer="19" extent="1-1"/>
@@
 <wire x1="6.29375" y1="20.32" x2="10.182" y2="22.53" width="0" layer="19" extent="1-1"/>
 <wire x1="23.1775" y1="11.90625" x2="17.758" y2="12.53" width="0" layer="19" extent="1-1"/>
-<wire x1="6.6675" y1="3.54875" x2="6.6675" y2="9.945" width="0" layer="19" extent="1-1"/>
+<wire x1="6.6675" y1="3.54875" x2="6.19125" y2="9.945" width="0" layer="19" extent="1-1"/>
 </signal>
 <signal name="SO1">
@@
 <contactref element="IC1" pad="10"/>
 <contactref element="C9" pad="2"/>
-<wire x1="6.6675" y1="18.3125" x2="7.385" y2="19.03" width="0.3302" layer="1"/>
-<wire x1="7.385" y1="19.03" x2="10.182" y2="19.03" width="0.3302" layer="1"/>
+<wire x1="6.19125" y1="18.3125" x2="6.90875" y2="19.03" width="0.3302" layer="1"/>
+<wire x1="6.90875" y1="19.03" x2="10.182" y2="19.03" width="0.3302" layer="1"/>
 </signal>
 <signal name="N$34">
 <contactref element="IC1" pad="11"/>
 <contactref element="C9" pad="1"/>
-<wire x1="6.6675" y1="16.6125" x2="8.585" y2="18.53" width="0.3302" layer="1"/>
-<wire x1="8.585" y1="18.53" x2="10.182" y2="18.53" width="0.3302" layer="1"/>
+<wire x1="6.19125" y1="16.6125" x2="8.10875" y2="18.53" width="0.3302" layer="1"/>
+<wire x1="8.10875" y1="18.53" x2="10.182" y2="18.53" width="0.3302" layer="1"/>
 </signal>
 <signal name="N$43">
 <contactref element="IC1" pad="19"/>
 <contactref element="DVDD_CAP" pad="2"/>
-<wire x1="10.182" y1="14.53" x2="7.11625" y2="14.53" width="0.381" layer="1"/>
-<wire x1="7.11625" y1="14.53" x2="6.6675" y2="14.97875" width="0.381" layer="1"/>
+<wire x1="10.182" y1="14.53" x2="6.64" y2="14.53" width="0.381" layer="1"/>
+<wire x1="6.64" y1="14.53" x2="6.19125" y2="14.97875" width="0.381" layer="1"/>
 </signal>
 <signal name="N$47">
@@
 <contactref element="AVDD_CAP" pad="1"/>
 <wire x1="10.182" y1="12.53" x2="9.36625" y2="12.53" width="0.3302" layer="1"/>
-<wire x1="6.6675" y1="11.645" x2="7.5859" y2="12.5634" width="0.4318" layer="1"/>
-<wire x1="7.5859" y1="12.5634" x2="9.24024375" y2="12.5634" width="0.4318" layer="1"/>
+<wire x1="6.19125" y1="11.645" x2="7.10965" y2="12.5634" width="0.4318" layer="1"/>
+<wire x1="7.10965" y1="12.5634" x2="9.24024375" y2="12.5634" width="0.4318" layer="1"/>
 <wire x1="9.24024375" y1="12.5634" x2="9.36625" y2="12.53" width="0" layer="19" extent="1-1"/>
 </signal>

Commit message: Ready for autoroutering (Tester) 4
Parts:
- moved VIN 2.25 mm to (12.7, 3.02), turned to 0 degrees
- moved AVDD_CAP 0.48 mm to (6.67, 10.8)
- moved C9 0.48 mm to (6.67, 17.5)
- moved DVDD_CAP 0.48 mm to (6.67, 14.1)
- moved C14 0.16 mm to (13.7, 6.83), turned to 180 degrees
- turned C15 to 180 degrees
Routing:
- net GND: track 51.8 -> 23.9 mm, vias 9 -> 0

Commit message: Ready for autoroutering (Tester) 5
Routing:
- net GND: track 23.9 -> 34.0 mm
Changed lines of the file:
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@@
 <wire x1="12.573" y1="6.59675" x2="12.8025" y2="6.82625" width="0.635" layer="1"/>
 <wire x1="12.8025" y1="6.82625" x2="12.8025" y2="8.41375" width="0.635" layer="1"/>
-<wire x1="12.8025" y1="8.41375" x2="12.8025" y2="12.64375" width="0.635" layer="1"/>
+<wire x1="12.8025" y1="8.41375" x2="12.8025" y2="11.43" width="0.635" layer="1"/>
+<wire x1="12.8025" y1="11.43" x2="12.8025" y2="12.64375" width="0.635" layer="1"/>
 <wire x1="12.8025" y1="12.64375" x2="12.85875" y2="12.7" width="0.635" layer="1"/>
+<wire x1="12.8025" y1="11.43" x2="12.3375" y2="11.895" width="0.635" layer="1"/>
+<wire x1="12.3375" y1="11.895" x2="10.16" y2="11.895" width="0.635" layer="1"/>
+<wire x1="12.8025" y1="12.64375" x2="12.8025" y2="16.6125" width="0.635" layer="1"/>
+<wire x1="12.8025" y1="16.6125" x2="13.97" y2="17.78" width="0.635" layer="1"/>
+<wire x1="17.758" y1="14.53" x2="16.2675" y2="14.53" width="0.3302" layer="1"/>
+<wire x1="16.2675" y1="14.53" x2="16.1925" y2="14.605" width="0.3302" layer="1"/>
 <wire x1="21.11375" y1="33.262" x2="23.01875" y2="33.262" width="0" layer="19" extent="1-1"/>
 <wire x1="17.758" y1="23.53" x2="21.11375" y2="33.262" width="0" layer="19" extent="1-1"/>
-<wire x1="17.758" y1="14.53" x2="17.758" y2="13.53" width="0" layer="19" extent="1-1"/>
 <wire x1="6.29375" y1="20.32" x2="10.182" y2="22.53" width="0" layer="19" extent="1-1"/>
 <wire x1="23.1775" y1="11.90625" x2="17.758" y2="12.53" width="0" layer="19" extent="1-1"/>
@@
 <wire x1="16.45553125" y1="11.895" x2="16.46823125" y2="11.9077" width="0.635" layer="1"/>
 <wire x1="16.46823125" y1="11.9077" x2="17.758" y2="11.9077" width="0.635" layer="1"/>
-<wire x1="17.758" y1="12.03" x2="17.758" y2="11.9736" width="0" layer="19" extent="1-1"/>
+<wire x1="17.758" y1="11.9736" x2="17.758" y2="12.03" width="0" layer="19" extent="1-1"/>
 <wire x1="17.758" y1="11.9077" x2="17.758" y2="11.9736" width="0" layer="19" extent="1-1"/>
 </signal>
