File: V4/Circuit/Driver.sch (EAGLE design)
At the start: 54 parts, among them IC1 DRV8303DCA

Commit message: Exported V4 circuit
Parts:
- added ENCODER: (no value), con-lstb:MA06-1
- added SERIAL: (no value), con-lstb:MA04-1
Connections:
- removed net PA0: U$1.PA0
- removed net PA1: U$1.PA1
- new net PA11: ENCODER.6, U$1.PA11
- new net PA12: ENCODER.5, U$1.PA12
- net 3V3: now also ENCODER.1, SERIAL.1
- net GND: now also ENCODER.2, ENCODER.3, SERIAL.2
- net PA15: now also ENCODER.4
- net PA2: now also SERIAL.3
- net PA3: now also SERIAL.4
- net SO1: now also U$1.PA1; no longer U$1.PA11
- net SO2: now also U$1.PA0; no longer U$1.PA12
Changed lines of the file:
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@@
 <part name="BUCK_CAP_B" library="SparkFun-Capacitors" deviceset="2.2UF" device="-0603-10V-20%" value="2.2uF"/>
 <part name="BUCK_CAP_C" library="SparkFun-Capacitors" deviceset="2.2UF" device="-0603-10V-20%" value="2.2uF"/>
+<part name="SERIAL" library="con-lstb" library_urn="urn:adsk.eagle:library:162" deviceset="MA04-1" device="" package3d_urn="urn:adsk.eagle:package:8337/1"/>
+<part name="SUPPLY27" library="supply2" library_urn="urn:adsk.eagle:library:372" deviceset="GND" device=""/>
+<part name="ENCODER" library="con-lstb" library_urn="urn:adsk.eagle:library:162" deviceset="MA06-1" device="" package3d_urn="urn:adsk.eagle:package:8340/1"/>
+<part name="SUPPLY28" library="supply2" library_urn="urn:adsk.eagle:library:372" deviceset="GND" device=""/>
+<part name="SUPPLY29" library="supply2" library_urn="urn:adsk.eagle:library:372" deviceset="GND" device=""/>
 </parts>
 <sheets>
@@
 <attribute name="VALUE" x="252.984" y="28.321" size="1.778" layer="96" font="vector"/>
 </instance>
+<instance part="SERIAL" gate="1" x="35.56" y="63.5" smashed="yes">
+<attribute name="VALUE" x="34.29" y="53.34" size="1.778" layer="96"/>
+<attribute name="NAME" x="34.29" y="69.342" size="1.778" layer="95"/>
+</instance>
+<instance part="SUPPLY27" gate="GND" x="53.34" y="60.96" smashed="yes" rot="R90">
+<attribute name="VALUE" x="56.515" y="59.055" size="1.778" layer="96" rot="R90"/>
+</instance>
+<instance part="ENCODER" gate="1" x="66.04" y="60.96" smashed="yes">
+<attribute name="VALUE" x="64.77" y="48.26" size="1.778" layer="96"/>
+<attribute name="NAME" x="64.77" y="69.342" size="1.778" layer="95"/>
+</instance>
+<instance part="SUPPLY28" gate="GND" x="86.36" y="58.42" smashed="yes" rot="R90">
+<attribute name="VALUE" x="89.535" y="56.515" size="1.778" layer="96" rot="R90"/>
+</instance>
+<instance part="SUPPLY29" gate="GND" x="86.36" y="55.88" smashed="yes" rot="R90">
+<attribute name="VALUE" x="89.535" y="53.975" size="1.778" layer="96" rot="R90"/>
+</instance>
 </instances>
 <busses>
@@
 <pinref part="SHUNT_CAP_A" gate="G$1" pin="2"/>
 <wire x1="190.5" y1="-22.86" x2="190.5" y2="-25.4" width="0.1524" layer="91"/>
+<junction x="195.58" y="-25.4"/>
 </segment>
 <segment>
@@
 <pinref part="SHUNT_CAP_B" gate="G$1" pin="2"/>
 <wire x1="215.9" y1="-22.86" x2="215.9" y2="-25.4" width="0.1524" layer="91"/>
+<junction x="220.98" y="-25.4"/>
 </segment>
 <segment>
@@
 <wire x1="246.38" y1="-12.7" x2="241.3" y2="-12.7" width="0.1524" layer="91"/>
 <label x="241.3" y="-12.7" size="1.27" layer="95" rot="R180" xref="yes"/>
+<junction x="246.38" y="-12.7"/>
 </segment>
 <segment>
@@
 <pinref part="BUCK_CAP_C" gate="G$1" pin="2"/>
 </segment>
+<segment>
+<pinref part="SERIAL" gate="1" pin="2"/>
+<pinref part="SUPPLY27" gate="GND" pin="GND"/>
+<wire x1="43.18" y1="60.96" x2="50.8" y2="60.96" width="0.1524" layer="91"/>
+</segment>
+<segment>
+<pinref part="ENCODER" gate="1" pin="3"/>
+<wire x1="73.66" y1="58.42" x2="83.82" y2="58.42" width="0.1524" layer="91"/>
+<pinref part="SUPPLY28" gate="GND" pin="GND"/>
+</segment>
+<segment>
+<pinref part="ENCODER" gate="1" pin="2"/>
+<wire x1="73.66" y1="55.88" x2="83.82" y2="55.88" width="0.1524" layer="91"/>
+<pinref part="SUPPLY29" gate="GND" pin="GND"/>
+</segment>
 </net>
 <net name="N$4" class="0">
@@
 <label x="88.9" y="96.52" size="1.27" layer="95" xref="yes"/>
 </segment>
+<segment>
+<pinref part="SERIAL" gate="1" pin="4"/>
+<wire x1="43.18" y1="66.04" x2="45.72" y2="66.04" width="0.1524" layer="91"/>
+<label x="45.72" y="66.04" size="1.27" layer="95" xref="yes"/>
+</segment>
 </net>
 <net name="PA2" class="0">
@@
 <label x="88.9" y="93.98" size="1.27" layer="95" xref="yes"/>
 </segment>
-</net>
-<net name="PA1" class="0">
-<segment>
-<pinref part="U$1" gate="G$1" pin="PA1"/>
-<wire x1="83.82" y1="91.44" x2="88.9" y2="91.44" width="0.1524" layer="91"/>
-<label x="88.9" y="91.44" size="1.27" layer="95" xref="yes"/>
-</segment>
-</net>
-<net name="PA0" class="0">
-<segment>
-<pinref part="U$1" gate="G$1" pin="PA0"/>
-<wire x1="83.82" y1="88.9" x2="88.9" y2="88.9" width="0.1524" layer="91"/>
-<label x="88.9" y="88.9" size="1.27" layer="95" xref="yes"/>
+<segment>
+<pinref part="SERIAL" gate="1" pin="3"/>
+<wire x1="43.18" y1="63.5" x2="45.72" y2="63.5" width="0.1524" layer="91"/>
+<label x="45.72" y="63.5" size="1.27" layer="95" xref="yes"/>
 </segment>
 </net>
@@
 <label x="38.1" y="104.14" size="1.27" layer="95" rot="R180" xref="yes"/>
 </segment>
+<segment>
+<pinref part="ENCODER" gate="1" pin="4"/>
+<wire x1="73.66" y1="60.96" x2="76.2" y2="60.96" width="0.1524" layer="91"/>
+<label x="76.2" y="60.96" size="1.27" layer="95" xref="yes"/>
+</segment>
 </net>
 <net name="PB3" class="0">
@@
 <wire x1="248.92" y1="83.82" x2="246.38" y2="83.82" width="0.1524" layer="91"/>
 <label x="246.38" y="83.82" size="1.27" layer="95" rot="R180" xref="yes"/>
+</segment>
+<segment>
+<pinref part="SERIAL" gate="1" pin="1"/>
+<wire x1="43.18" y1="58.42" x2="45.72" y2="58.42" width="0.1524" layer="91"/>
+<label x="45.72" y="58.42" size="1.27" layer="95" xref="yes"/>
+</segment>
+<segment>
+<pinref part="ENCODER" gate="1" pin="1"/>
+<wire x1="73.66" y1="53.34" x2="76.2" y2="53.34" width="0.1524" layer="91"/>
+<label x="76.2" y="53.34" size="1.27" layer="95" xref="yes"/>
 </segment>
 </net>
@@
 <pinref part="SHUNT_CAP_A" gate="G$1" pin="1"/>
 <wire x1="190.5" y1="-15.24" x2="190.5" y2="-12.7" width="0.1524" layer="91"/>
+<junction x="195.58" y="-12.7"/>
 </segment>
 <segment>
@@
 <pinref part="SHUNT_CAP_B" gate="G$1" pin="1"/>
 <wire x1="215.9" y1="-15.24" x2="215.9" y2="-12.7" width="0.1524" layer="91"/>
+<junction x="220.98" y="-12.7"/>
 </segment>
 <segment>
@@
 <wire x1="200.66" y1="38.1" x2="200.66" y2="35.56" width="0.1524" layer="91"/>
 <pinref part="BUCK_CAP_A" gate="G$1" pin="1"/>
+<junction x="195.58" y="38.1"/>
 </segment>
 <segment>
@@
 <wire x1="226.06" y1="38.1" x2="226.06" y2="35.56" width="0.1524" layer="91"/>
 <pinref part="BUCK_CAP_B" gate="G$1" pin="1"/>
+<junction x="220.98" y="38.1"/>
 </segment>
 <segment>
@@
 <wire x1="251.46" y1="38.1" x2="251.46" y2="35.56" width="0.1524" layer="91"/>
 <pinref part="BUCK_CAP_C" gate="G$1" pin="1"/>
+<junction x="246.38" y="38.1"/>
 </segment>
 <segment>
@@
 <wire x1="246.38" y1="132.08" x2="246.38" y2="139.7" width="0.1524" layer="91"/>
 <pinref part="R3" gate="G$1" pin="1"/>
+<junction x="246.38" y="132.08"/>
 </segment>
 <segment>
@@
 <net name="SO1" class="0">
 <segment>
-<pinref part="U$1" gate="G$1" pin="PA11"/>
-<wire x1="43.18" y1="109.22" x2="38.1" y2="109.22" width="0.1524" layer="91"/>
-<label x="38.1" y="109.22" size="1.27" layer="95" rot="R180" xref="yes"/>
-</segment>
-<segment>
 <wire x1="236.22" y1="81.28" x2="233.68" y2="81.28" width="0.1524" layer="91"/>
 <label x="233.68" y="81.28" size="1.27" layer="95" rot="R180" xref="yes"/>
 <pinref part="R5" gate="R1" pin="1"/>
 </segment>
+<segment>
+<pinref part="U$1" gate="G$1" pin="PA1"/>
+<wire x1="83.82" y1="91.44" x2="88.9" y2="91.44" width="0.1524" layer="91"/>
+<label x="88.9" y="91.44" size="1.27" layer="95" xref="yes"/>
+</segment>
 </net>
 <net name="SO2" class="0">
-<segment>
-<pinref part="U$1" gate="G$1" pin="PA12"/>
-<wire x1="43.18" y1="106.68" x2="38.1" y2="106.68" width="0.1524" layer="91"/>
-<label x="38.1" y="106.68" size="1.27" layer="95" rot="R180" xref="yes"/>
-</segment>
 <segment>
 <wire x1="236.22" y1="78.74" x2="233.68" y2="78.74" width="0.1524" layer="91"/>
 <label x="233.68" y="78.74" size="1.27" layer="95" rot="R180" xref="yes"/>
 <pinref part="R6" gate="R1" pin="1"/>
+</segment>
+<segment>
+<pinref part="U$1" gate="G$1" pin="PA0"/>
+<wire x1="83.82" y1="88.9" x2="88.9" y2="88.9" width="0.1524" layer="91"/>
+<label x="88.9" y="88.9" size="1.27" layer="95" xref="yes"/>
 </segment>
 </net>
@@
 </segment>
 </net>
+<net name="PA11" class="0">
+<segment>
+<pinref part="U$1" gate="G$1" pin="PA11"/>
+<wire x1="43.18" y1="109.22" x2="38.1" y2="109.22" width="0.1524" layer="91"/>
+<label x="38.1" y="109.22" size="1.27" layer="95" rot="R180" xref="yes"/>
+</segment>
+<segment>
+<pinref part="ENCODER" gate="1" pin="6"/>
+<wire x1="73.66" y1="66.04" x2="76.2" y2="66.04" width="0.1524" layer="91"/>
+<label x="76.2" y="66.04" size="1.27" layer="95" xref="yes"/>
+</segment>
+</net>
+<net name="PA12" class="0">
+<segment>
+<pinref part="U$1" gate="G$1" pin="PA12"/>
+<wire x1="43.18" y1="106.68" x2="38.1" y2="106.68" width="0.1524" layer="91"/>
+<label x="38.1" y="106.68" size="1.27" layer="95" rot="R180" xref="yes"/>
+</segment>
+<segment>
+<pinref part="ENCODER" gate="1" pin="5"/>
+<wire x1="73.66" y1="63.5" x2="76.2" y2="63.5" width="0.1524" layer="91"/>
+<label x="76.2" y="63.5" size="1.27" layer="95" xref="yes"/>
+</segment>
+</net>
